File: m2r1/WaveSL.kicad_pcb (KiCad board)
At the start: 4 copper layers, 55 x 20 mm, 42 parts, among them J1 Screw_Terminal_01x02, J2 SOICBite, U1 LED2000DR, U2 LMZM23600V3SILR, U3 MPL3115A2, U4 LM75BTP, U5 LPC812M001JDH16

Commit message: cleanup F.Fab and add IBOM
Parts:
- R2: value R -> 1k5
- R3, R4: value R -> 270R
- R5, R6, R7, R8: value R -> 10k
- R9: value R -> 0R
